File: robotarna_arduino.sch (KiCad schematic (older format))
At the start: 65 parts, among them P1 CONN_01X02, P10 CONN_01X02, P11 CONN_01X02, P12 CONN_01X02, P13 CONN_01X02, P14 DHT11_CONN, P15 CONN_01X02, P16 CONN_01X02, P2 CONN_01X02, P3 CONN_01X02, P4 CONN_01X02, P5 CONN_01X02, P6 CONN_01X02, P7 CONN_01X02, P8 CONN_01X02, P9 CONN_01X02, U1 arduino_nano, U2 arduino_uno, U3 PIEZO

Commit message: Add some routing and remove jumpers
Parts:
- removed P1, P10, P11, P12, P13, P15, P16, P2, P3, P4, P5, P6, P7, P8, P9: CONN_01X02, Pin_Headers:Pin_Header_Straight_1x02, symbol CONN_01X02
- RV1: footprint Resistors_SMD:R_1206_HandSoldering -> Potentiometers:RV09
- RV2: footprint Resistors_SMD:R_1210 -> Potentiometers:RV09
- SW1, SW2, SW3: renamed from SW?; footprint (none) -> Buttons_Switches_ThroughHole:SW_PUSH_6mm
Connections:
- wire segments 96 -> 44

Commit message: Final version for production
Parts:
- C1, C2, C3: symbol C -> C-RESCUE-robotarna_arduino
- R1, R10, R11, R12, R13, R14, R15, R16, R17, R18, R2, R4, R5, R6, R7, R8, R9: symbol R -> R-RESCUE-robotarna_arduino
Changed lines of the file:
@@
 EESchema Schematic File Version 2
-LIBS:Zilog
-LIBS:xilinx
-LIBS:Xicor
-LIBS:Worldsemi
-LIBS:video
-LIBS:valves
-LIBS:ttl_ieee
-LIBS:transistors
-LIBS:transf
-LIBS:texas
-LIBS:switches
-LIBS:supertex
-LIBS:stm32
-LIBS:stm8
-LIBS:siliconi
-LIBS:silabs
-LIBS:sensors
-LIBS:rfcom
-LIBS:relays
-LIBS:regul
-LIBS:references
-LIBS:pspice
+LIBS:robotarna_arduino-rescue
+LIBS:74xgxx
+LIBS:74xx
+LIBS:ac-dc
+LIBS:actel
+LIBS:adc-dac
+LIBS:Altera
+LIBS:analog_devices
+LIBS:analog_switches
+LIBS:atmel
+LIBS:audio
+LIBS:battery_management
+LIBS:bbd
+LIBS:brooktre
+LIBS:cmos_ieee
+LIBS:cmos4000
+LIBS:conn
+LIBS:contrib
+LIBS:cypress
+LIBS:dc-dc
+LIBS:device
+LIBS:digital-audio
+LIBS:diode
+LIBS:display
+LIBS:dsp
+LIBS:elec-unifil
+LIBS:ESD_Protection
+LIBS:ftdi
+LIBS:gennum
+LIBS:graphic
+LIBS:hc11
+LIBS:intel
+LIBS:interface
+LIBS:ir
+LIBS:Lattice
+LIBS:linear
+LIBS:logo
+LIBS:maxim
+LIBS:memory
+LIBS:microcontrollers
+LIBS:microchip
+LIBS:microchip_dspic33dsc
+LIBS:microchip_pic10mcu
+LIBS:microchip_pic12mcu
+LIBS:microchip_pic16mcu
+LIBS:microchip_pic18mcu
+LIBS:microchip_pic32mcu
+LIBS:motor_drivers
+LIBS:motorola
+LIBS:msp430
+LIBS:nordicsemi
+LIBS:nxp_armmcu
+LIBS:onsemi
+LIBS:opto
+LIBS:Oscillators
+LIBS:philips
+LIBS:power
 LIBS:Power_Management
 LIBS:powerint
-LIBS:power
-LIBS:philips
-LIBS:Oscillators
-LIBS:opto
-LIBS:onsemi
-LIBS:nxp_armmcu
-LIBS:nordicsemi
-LIBS:msp430
-LIBS:motorola
-LIBS:motor_drivers
-LIBS:microchip_pic32mcu
-LIBS:microchip_pic18mcu
-LIBS:microchip_pic16mcu
-LIBS:microchip_pic12mcu
-LIBS:microchip_pic10mcu
-LIBS:microchip_dspic33dsc
-LIBS:microchip
-LIBS:microcontrollers
-LIBS:memory
-LIBS:maxim
-LIBS:logo
-LIBS:linear
-LIBS:Lattice
-LIBS:ir
-LIBS:interface
-LIBS:intel
-LIBS:hc11
-LIBS:graphic
-LIBS:gennum
-LIBS:ftdi
-LIBS:ESD_Protection
-LIBS:elec-unifil
-LIBS:dsp
-LIBS:display
-LIBS:diode
-LIBS:digital-audio
-LIBS:device
-LIBS:dc-dc
-LIBS:cypress
-LIBS:contrib
-LIBS:conn
-LIBS:cmos_ieee
-LIBS:cmos4000
-LIBS:brooktre
-LIBS:bbd
-LIBS:battery_management
-LIBS:audio
-LIBS:atmel
-LIBS:analog_switches
-LIBS:analog_devices
-LIBS:Altera
-LIBS:adc-dac
-LIBS:actel
-LIBS:ac-dc
-LIBS:74xx
-LIBS:74xgxx
-LIBS:shield_arduino
-LIBS:yaqwsx
+LIBS:pspice
+LIBS:references
+LIBS:regul
+LIBS:relays
+LIBS:rfcom
+LIBS:sensors
+LIBS:silabs
+LIBS:siliconi
+LIBS:stm8
+LIBS:stm32
+LIBS:supertex
+LIBS:switches
+LIBS:texas
+LIBS:transf
+LIBS:transistors
+LIBS:ttl_ieee
+LIBS:valves
+LIBS:video
+LIBS:Worldsemi
+LIBS:Xicor
+LIBS:xilinx
+LIBS:Zilog
 LIBS:robotarna_arduino-cache
 EELAYER 25 0
@@
 $EndComp
 $Comp
-L R R16
+L R-RESCUE-robotarna_arduino R16
 U 1 1 57E2FB4D
 P 9000 3450
@@
 $EndComp
 $Comp
-L R R17
+L R-RESCUE-robotarna_arduino R17
 U 1 1 57E2FBFC
 P 9000 3650
@@
 $EndComp
 $Comp
-L R R18
+L R-RESCUE-robotarna_arduino R18
 U 1 1 57E2FC45
 P 9000 3850
@@
 $EndComp
 $Comp
-L R R8
+L R-RESCUE-robotarna_arduino R8
 U 1 1 57E354F8
 P 4350 4950
@@
 $EndComp
 $Comp
-L R R9
+L R-RESCUE-robotarna_arduino R9
 U 1 1 57E35DE4
 P 4350 5600
@@
 $EndComp
 $Comp
-L R R5
+L R-RESCUE-robotarna_arduino R5
 U 1 1 57E36617
 P 4300 6250
@@
 $EndComp
 $Comp
-L R R6
+L R-RESCUE-robotarna_arduino R6
 U 1 1 57E3663A
 P 4300 6900
@@
 	1500 6500 2050 6500
 $Comp
-L R R4
+L R-RESCUE-robotarna_arduino R4
 U 1 1 57E37C7D
 P 2050 6750
@@
 	9550 3450 9600 3450
 $Comp
-L R R7
+L R-RESCUE-robotarna_arduino R7
 U 1 1 57E30046
 P 4350 4100
@@
 	4700 4100 4600 4100
 $Comp
-L R R1
+L R-RESCUE-robotarna_arduino R1
 U 1 1 57E44C39
 P 1800 4150
@@
 A1
 $Comp
-L R R2
+L R-RESCUE-robotarna_arduino R2
 U 1 1 57E4524A
 P 1800 5150
@@
 $EndComp
 $Comp
-L C C3
+L C-RESCUE-robotarna_arduino C3
 U 1 1 57E46232
 P 6950 3000
@@
 $EndComp
 $Comp
-L R R15
+L R-RESCUE-robotarna_arduino R15
 U 1 1 57E468B0
 P 6350 3450
@@
 $EndComp
 $Comp
-L C C1
+L C-RESCUE-robotarna_arduino C1
 U 1 1 57E479A1
 P 6900 4200
@@
 $EndComp
 $Comp
-L R R13
+L R-RESCUE-robotarna_arduino R13
 U 1 1 57E479AD
 P 6300 4650
@@
 $EndComp
 $Comp
-L C C2
+L C-RESCUE-robotarna_arduino C2
 U 1 1 57E47D71
 P 6900 5450
@@
 $EndComp
 $Comp
-L R R14
+L R-RESCUE-robotarna_arduino R14
 U 1 1 57E47D7D
 P 6300 5900
@@
 Connection ~ 6550 5900
 $Comp
-L R R12
+L R-RESCUE-robotarna_arduino R12
 U 1 1 57E48021
 P 6100 3700
@@
 $EndComp
 $Comp
-L R R10
+L R-RESCUE-robotarna_arduino R10
 U 1 1 57E4856A
 P 6050 4900
@@
 $EndComp
 $Comp
-L R R11
+L R-RESCUE-robotarna_arduino R11
 U 1 1 57E48844
 P 6050 6150

Commit message: Fix labels (#close 6)
Parts:
- L_B: renamed from D4; symbol LED -> LED-RESCUE-robotarna_arduino
- L_G: renamed from D3; symbol LED -> LED-RESCUE-robotarna_arduino
- L_R: renamed from D1; symbol LED -> LED-RESCUE-robotarna_arduino
- L_RGB: renamed from D5; symbol LED_RCBG -> LED_RCBG-RESCUE-robotarna_arduino
- L_Y: renamed from D2; symbol LED -> LED-RESCUE-robotarna_arduino
- RV1, RV2: symbol POT -> POT-RESCUE-robotarna_arduino
- renumbered P14 to DHT11, R3 to PHOTO1, U3 to PIEIZO1

Commit message: Initial commit for version 2
Parts:
- added J1: USB_OTG, yaqwsx:USB_Micro-B-widened, symbol USB_OTG
- added J2, J4: CONN_01X08, yaqwsx:Pin_Header_Straight_1x08_circle, symbol CONN_01X08
- added J3: CONN_01X06, yaqwsx:Pin_Header_Straight_1x06_circle, symbol CONN_01X06
- added J5: CONN_01X10, yaqwsx:Pin_Header_Straight_1x10_circle, symbol CONN_01X10
- added JP16: Jumper, Pin_Headers:Pin_Header_Straight_1x02, symbol Jumper_NC_Small
- added R19, R20, R21, R22, R3: 1k, Resistors_SMD:R_1206_HandSoldering, symbol R
- added S1: SERVO1, Pin_Headers:Pin_Header_Straight_1x03, symbol CONN_01X03
- added S2: SERVO2, Pin_Headers:Pin_Header_Straight_1x03, symbol CONN_01X03
- added S3: SERVO3, Pin_Headers:Pin_Header_Straight_1x03, symbol CONN_01X03
- added S4: SERVO4, Pin_Headers:Pin_Header_Straight_1x03, symbol CONN_01X03
- added S5: SERVO5, Pin_Headers:Pin_Header_Straight_1x03, symbol CONN_01X03
- JP9: value Jumper_NC_Small -> Jumper; footprint yaqwsx:CUT_BRIDGGE -> Pin_Headers:Pin_Header_Straight_1x02
- U2: footprint yaqwsx:arduino_uno -> yaqwsx:arduino_uno_small_pads
- renumbered L_B to L_B1, L_G to L_G1, L_R to L_R1, L_RGB to L_RGB1, L_Y to L_Y1
Connections:
- net +3V3: now also J2.4 (P4)
- net +5V: now also JP9.1, J2.5 (P5), J2.6 (P6), J2.7 (P7), J2.8 (P8)
- net D10: now also JP16.2, R21.1; no longer JP9.2
- net D11: now also R22.1
- net D5: now also R3.1
- net D6: now also R19.1
- net D9: now also R20.1
- net GND: now also J1.5 (GND), J1.6 (Shield), J2.1 (P1), J2.3 (P3), J3.1 (P1), J3.2 (P2), J3.3 (P3), J3.4 (P4), J3.5 (P5), J3.6 (P6), J4.1 (P1), J4.2 (P2), J4.3 (P3), J4.4 (P4), J4.5 (P5), J4.6 (P6), J4.7 (P7), J4.8 (P8), J5.1 (P1), J5.10 (P10), J5.2 (P2), J5.3 (P3), J5.4 (P4), J5.5 (P5), J5.6 (P6), J5.7 (P7), J5.8 (P8), J5.9 (P9), S1.1 (P1), S2.1 (P1), S3.1 (P1), S4.1 (P1), S5.1 (P1)
- net IOREF: now reaches U2.2 (IOREF)
- net IOREF: now also J2.2 (P2)
- net at R7.1: now also JP16.1; no longer JP9.1
- new net: R3.2, S1.3 (P3)
- new net: R19.2, S2.3 (P3)
- new net: R20.2, S3.3 (P3)
- new net: R21.2, S4.3 (P3)
- new net: R22.2, S5.3 (P3)
- new net VCC_SERVO: J1.1 (VBUS), JP9.2, S1.2 (P2), S2.2 (P2), S3.2 (P2), S4.2 (P2), S5.2 (P2)
- no-connect marks 3 -> 5
Other:
- moved on the sheet: C1, C2, C3, DHT11, JP1, JP10, JP11, JP12, JP13, JP14, JP15, JP2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

Commit message: Final version of schematics
Parts:
- added J6, J7: CONN_01X04, Pin_Headers:Pin_Header_Straight_1x04, symbol CONN_01X04
- added JP17: Jumper, Pin_Headers:Pin_Header_Straight_1x02, symbol Jumper_NC_Small
- added R23, R24: 1k, Resistors_SMD:R_1206_HandSoldering, symbol R
- added R25: 20k, Resistors_SMD:R_1206_HandSoldering, symbol R
Connections:
- net +5V: now also J6.4 (P4), J7.4 (P4)
- net A3: now also J7.3 (P3)
- net D0: now also R23.1
- net D1: now also R24.1
- net D2: now also JP10.1; no longer JP12.1
- net D3: now also JP11.1; no longer JP10.1
- net D4: now also JP12.1; no longer JP11.1
- net GND: now also J6.3 (P3), J7.1 (P1), R25.1
- net at R13.1, SW1.1: now also JP17.1; no longer C1.2
- net at JP10.2, R13.2: no longer R10.2
- new net: C1.2, JP17.2, R10.2
- new net: J6.1 (P1), R24.2
- new net: J6.2 (P2), R23.2
- new net: J7.2 (P2), R25.2
Other:
- moved on the sheet: C1, C2, C3, JP10, JP11, JP12, R10, R11, R12, R13, R14, R15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

Commit message: Add labels, mouting holes, repair some mistakes and tracks
Parts:
- J1: symbol USB_OTG -> USB_OTG-RESCUE-robotarna_arduino
- R19, R20, R21, R22, R23, R24: symbol R -> R-RESCUE-robotarna_arduino
- R25: renamed from R3; symbol R -> R-RESCUE-robotarna_arduino
- R3: renamed from R25; symbol R -> R-RESCUE-robotarna_arduino
