File: ArduinoLearningKitStarter.sch (KiCad schematic (older format))
At the start: 72 parts, among them J1 USB_OTG, J2 CONN_01X08, J3 CONN_01X06, J4 CONN_01X08, J5 CONN_01X10, J6 CONN_01X04, J7 CONN_01X04, SW1 SW_PUSH, SW2 SW_PUSH, SW3 SW_PUSH, U1 arduino_nano, U2 arduino_uno

Commit message: Repair problem in schema with ArduinoLearningKitStarter-rescue.lib
Parts:
- J1: symbol USB_OTG-RESCUE-robotarna_arduino -> USB_OTG
Connections:
- wire segments 63 -> 87
Changed lines of the file:
@@
 EESchema Schematic File Version 2
-LIBS:robotarna_arduino-rescue
+LIBS:ArduinoLearningKitStarter-rescue
 LIBS:74xgxx
 LIBS:74xx
@@
 LIBS:xilinx
 LIBS:Zilog
-LIBS:robotarna_arduino-cache
 EELAYER 25 0
 EELAYER END
@@
 $EndComp
 $Comp
-L USB_OTG-RESCUE-robotarna_arduino J1
+L USB_OTG J1
 U 1 1 58C23B71
 P 1150 6750
@@
 	9050 4850 9050 5300
 Wire Wire Line
-	9000 5300 9150 5300
+	9000 5300 9050 5300
+Wire Wire Line
+	9050 5300 9150 5300
 Connection ~ 9050 5300
 Connection ~ 8400 5300
@@
 	9050 3050 9050 3500
 Wire Wire Line
-	9000 3500 9150 3500
+	9000 3500 9050 3500
+Wire Wire Line
+	9050 3500 9150 3500
 Connection ~ 9050 3500
 Connection ~ 8400 3500
@@
 	9050 3850 9050 4300
 Wire Wire Line
-	9000 4300 9150 4300
+	9000 4300 9050 4300
+Wire Wire Line
+	9050 4300 9150 4300
 Connection ~ 9050 4300
 Connection ~ 8400 4300
@@
 	1650 6300 1650 6550
 Wire Wire Line
-	1450 6550 1750 6550
+	1450 6550 1650 6550
+Wire Wire Line
+	1650 6550 1750 6550
 Connection ~ 1650 6550
 Connection ~ 4400 3750
@@
 Connection ~ 4400 3950
 Wire Wire Line
-	4400 4350 4400 4850
+	4400 4350 4400 4450
+Wire Wire Line
+	4400 4450 4400 4550
+Wire Wire Line
+	4400 4550 4400 4650
+Wire Wire Line
+	4400 4650 4400 4750
+Wire Wire Line
+	4400 4750 4400 4850
 Connection ~ 4400 4450
 Connection ~ 4400 4550
@@
 Connection ~ 4400 4750
 Wire Wire Line
-	4400 5150 4400 5850
+	4400 5150 4400 5250
+Wire Wire Line
+	4400 5250 4400 5350
+Wire Wire Line
+	4400 5350 4400 5450
+Wire Wire Line
+	4400 5450 4400 5550
+Wire Wire Line
+	4400 5550 4400 5650
+Wire Wire Line
+	4400 5650 4400 5750
+Wire Wire Line
+	4400 5750 4400 5850
 Connection ~ 4400 5250
 Connection ~ 4400 5350
@@
 Connection ~ 4400 5750
 Wire Wire Line
-	4400 6200 4400 7100
+	4400 6200 4400 6300
+Wire Wire Line
+	4400 6300 4400 6400
+Wire Wire Line
+	4400 6400 4400 6500
+Wire Wire Line
+	4400 6500 4400 6600
+Wire Wire Line
+	4400 6600 4400 6700
+Wire Wire Line
+	4400 6700 4400 6800
+Wire Wire Line
+	4400 6800 4400 6900
+Wire Wire Line
+	4400 6900 4400 7000
+Wire Wire Line
+	4400 7000 4400 7100
 Connection ~ 4400 6300
 Connection ~ 4400 6400
@@
 Connection ~ 4400 7000
 Wire Wire Line
-	4400 3750 4400 4050
+	4400 3750 4400 3850
+Wire Wire Line
+	4400 3850 4400 3950
+Wire Wire Line
+	4400 3950 4400 4050
 $Comp
 L GND #PWR042

Commit message: Add capacitors to servo connectors
Parts:
- added C4, C5, C6, C7, C8: C_Small, Capacitors_SMD:C_0805_HandSoldering, symbol C_Small
Connections:
- wire segments 87 -> 78
Changed lines of the file:
@@
 EESchema Schematic File Version 2
 LIBS:ArduinoLearningKitStarter-rescue
-LIBS:74xgxx
-LIBS:74xx
-LIBS:ac-dc
-LIBS:actel
-LIBS:adc-dac
-LIBS:Altera
-LIBS:analog_devices
-LIBS:analog_switches
-LIBS:atmel
-LIBS:audio
-LIBS:battery_management
-LIBS:bbd
-LIBS:brooktre
+LIBS:Zilog
+LIBS:xilinx
+LIBS:Xicor
+LIBS:Worldsemi
+LIBS:video
+LIBS:valves
+LIBS:ttl_ieee
+LIBS:transistors
+LIBS:transf
+LIBS:texas
+LIBS:switches
+LIBS:supertex
+LIBS:stm32
+LIBS:stm8
+LIBS:siliconi
+LIBS:silabs
+LIBS:sensors
+LIBS:rfcom
+LIBS:relays
+LIBS:regul
+LIBS:references
+LIBS:pspice
+LIBS:Power_Management
+LIBS:powerint
+LIBS:power
+LIBS:philips
+LIBS:Oscillators
+LIBS:opto
+LIBS:onsemi
+LIBS:nxp_armmcu
+LIBS:nordicsemi
+LIBS:msp430
+LIBS:motorola
+LIBS:motor_drivers
+LIBS:microchip_pic32mcu
+LIBS:microchip_pic18mcu
+LIBS:microchip_pic16mcu
+LIBS:microchip_pic12mcu
+LIBS:microchip_pic10mcu
+LIBS:microchip_dspic33dsc
+LIBS:microchip
+LIBS:microcontrollers
+LIBS:memory
+LIBS:maxim
+LIBS:logo
+LIBS:linear
+LIBS:Lattice
+LIBS:ir
+LIBS:interface
+LIBS:intel
+LIBS:hc11
+LIBS:graphic
+LIBS:gennum
+LIBS:ftdi
+LIBS:ESD_Protection
+LIBS:elec-unifil
+LIBS:dsp
+LIBS:display
+LIBS:diode
+LIBS:digital-audio
+LIBS:device
+LIBS:dc-dc
+LIBS:cypress
+LIBS:contrib
+LIBS:conn
 LIBS:cmos_ieee
 LIBS:cmos4000
-LIBS:conn
-LIBS:contrib
-LIBS:cypress
-LIBS:dc-dc
-LIBS:device
-LIBS:digital-audio
-LIBS:diode
-LIBS:display
-LIBS:dsp
-LIBS:elec-unifil
-LIBS:ESD_Protection
-LIBS:ftdi
-LIBS:gennum
-LIBS:graphic
-LIBS:hc11
-LIBS:intel
-LIBS:interface
-LIBS:ir
-LIBS:Lattice
-LIBS:linear
-LIBS:logo
-LIBS:maxim
-LIBS:memory
-LIBS:microcontrollers
-LIBS:microchip
-LIBS:microchip_dspic33dsc
-LIBS:microchip_pic10mcu
-LIBS:microchip_pic12mcu
-LIBS:microchip_pic16mcu
-LIBS:microchip_pic18mcu
-LIBS:microchip_pic32mcu
-LIBS:motor_drivers
-LIBS:motorola
-LIBS:msp430
-LIBS:nordicsemi
-LIBS:nxp_armmcu
-LIBS:onsemi
-LIBS:opto
-LIBS:Oscillators
-LIBS:philips
-LIBS:power
-LIBS:Power_Management
-LIBS:powerint
-LIBS:pspice
-LIBS:references
-LIBS:regul
-LIBS:relays
-LIBS:rfcom
-LIBS:sensors
-LIBS:silabs
-LIBS:siliconi
-LIBS:stm8
-LIBS:stm32
-LIBS:supertex
-LIBS:switches
-LIBS:texas
-LIBS:transf
-LIBS:transistors
-LIBS:ttl_ieee
-LIBS:valves
-LIBS:video
-LIBS:Worldsemi
-LIBS:Xicor
-LIBS:xilinx
-LIBS:Zilog
+LIBS:brooktre
+LIBS:bbd
+LIBS:battery_management
+LIBS:audio
+LIBS:atmel
+LIBS:analog_switches
+LIBS:analog_devices
+LIBS:Altera
+LIBS:adc-dac
+LIBS:actel
+LIBS:ac-dc
+LIBS:74xx
+LIBS:74xgxx
+LIBS:shield_arduino
+LIBS:yaqwsx
+LIBS:ArduinoLearningKitStarter-cache
 EELAYER 25 0
 EELAYER END
@@
 	9050 4850 9050 5300
 Wire Wire Line
-	9000 5300 9050 5300
-Wire Wire Line
-	9050 5300 9150 5300
+	9000 5300 9150 5300
 Connection ~ 9050 5300
 Connection ~ 8400 5300
@@
 	9050 3050 9050 3500
 Wire Wire Line
-	9000 3500 9050 3500
-Wire Wire Line
-	9050 3500 9150 3500
+	9000 3500 9150 3500
 Connection ~ 9050 3500
 Connection ~ 8400 3500
@@
 	9050 3850 9050 4300
 Wire Wire Line
-	9000 4300 9050 4300
-Wire Wire Line
-	9050 4300 9150 4300
+	9000 4300 9150 4300
 Connection ~ 9050 4300
 Connection ~ 8400 4300
@@
 	1650 6300 1650 6550
 Wire Wire Line
-	1450 6550 1650 6550
-Wire Wire Line
-	1650 6550 1750 6550
+	1450 6550 1750 6550
 Connection ~ 1650 6550
 Connection ~ 4400 3750
@@
 Connection ~ 4400 3950
 Wire Wire Line
-	4400 4350 4400 4450
-Wire Wire Line
-	4400 4450 4400 4550
-Wire Wire Line
-	4400 4550 4400 4650
-Wire Wire Line
-	4400 4650 4400 4750
-Wire Wire Line
-	4400 4750 4400 4850
+	4400 4350 4400 4850
 Connection ~ 4400 4450
 Connection ~ 4400 4550
@@
 Connection ~ 4400 4750
 Wire Wire Line
-	4400 5150 4400 5250
-Wire Wire Line
-	4400 5250 4400 5350
-Wire Wire Line
-	4400 5350 4400 5450
-Wire Wire Line
-	4400 5450 4400 5550
-Wire Wire Line
-	4400 5550 4400 5650
-Wire Wire Line
-	4400 5650 4400 5750
-Wire Wire Line
-	4400 5750 4400 5850
+	4400 5150 4400 5850
 Connection ~ 4400 5250
 Connection ~ 4400 5350
@@
 Connection ~ 4400 5750
 Wire Wire Line
-	4400 6200 4400 6300
-Wire Wire Line
-	4400 6300 4400 6400
-Wire Wire Line
-	4400 6400 4400 6500
-Wire Wire Line
-	4400 6500 4400 6600
-Wire Wire Line
-	4400 6600 4400 6700
-Wire Wire Line
-	4400 6700 4400 6800
-Wire Wire Line
-	4400 6800 4400 6900
-Wire Wire Line
-	4400 6900 4400 7000
-Wire Wire Line
-	4400 7000 4400 7100
+	4400 6200 4400 7100
 Connection ~ 4400 6300
 Connection ~ 4400 6400
@@
 Connection ~ 4400 7000
 Wire Wire Line
-	4400 3750 4400 3850
-Wire Wire Line
-	4400 3850 4400 3950
-Wire Wire Line
-	4400 3950 4400 4050
+	4400 3750 4400 4050
 $Comp
 L GND #PWR042
@@
 Text GLabel 7700 3500 0    60   Input ~ 0
 D2
+$Comp
+L C_Small C4
+U 1 1 58DE66DE
+P 1700 3800
+F 0 "C4" H 1710 3870 50  0000 L CNN
+F 1 "C_Small" H 1710 3720 50  0000 L CNN
+F 2 "Capacitors_SMD:C_0805_HandSoldering" H 1700 3800 50  0001 C CNN
+F 3 "" H 1700 3800 50  0001 C CNN
+	1    1700 3800
+	1    0    0    -1
+$EndComp
+Wire Wire Line
+	1200 3800 1450 3800
+Wire Wire Line
+	1450 3800 1450 3900
+Wire Wire Line
+	1450 3900 1700 3900
+$Comp
+L C_Small C5
+U 1 1 58DE6B28
+P 1700 4400
+F 0 "C5" H 1710 4470 50  0000 L CNN
+F 1 "C_Small" H 1710 4320 50  0000 L CNN
+F 2 "Capacitors_SMD:C_0805_HandSoldering" H 1700 4400 50  0001 C CNN
+F 3 "" H 1700 4400 50  0001 C CNN
+	1    1700 4400
+	1    0    0    -1
+$EndComp
+Wire Wire Line
+	1700 4500 1450 4500
+Wire Wire Line
+	1450 4500 1450 4400
+Wire Wire Line
+	1450 4400 1200 4400
+$Comp
+L C_Small C6
+U 1 1 58DE6CDD
+P 1700 4900
+F 0 "C6" H 1710 4970 50  0000 L CNN
+F 1 "C_Small" H 1710 4820 50  0000 L CNN
+F 2 "Capacitors_SMD:C_0805_HandSoldering" H 1700 4900 50  0001 C CNN
+F 3 "" H 1700 4900 50  0001 C CNN
+	1    1700 4900
+	1    0    0    -1
+$EndComp
+Wire Wire Line
+	1700 5000 1450 5000
+Wire Wire Line
+	1450 5000 1450 4900
+Wire Wire Line
+	1450 4900 1200 4900
+$Comp
+L C_Small C7
+U 1 1 58DE7055
+P 1700 5400
+F 0 "C7" H 1710 5470 50  0000 L CNN
+F 1 "C_Small" H 1710 5320 50  0000 L CNN
+F 2 "Capacitors_SMD:C_0805_HandSoldering" H 1700 5400 50  0001 C CNN
+F 3 "" H 1700 5400 50  0001 C CNN
+	1    1700 5400
+	1    0    0    -1
+$EndComp
+Wire Wire Line
+	1700 5500 1450 5500
+Wire Wire Line
+	1450 5500 1450 5400
+Wire Wire Line
+	1450 5400 1200 5400
+$Comp
+L C_Small C8
+U 1 1 58DE720C
+P 1900 5900
+F 0 "C8" H 1910 5970 50  0000 L CNN
+F 1 "C_Small" H 1910 5820 50  0000 L CNN
+F 2 "Capacitors_SMD:C_0805_HandSoldering" H 1900 5900 50  0001 C CNN
+F 3 "" H 1900 5900 50  0001 C CNN
+	1    1900 5900
+	1    0    0    -1
+$EndComp
+Wire Wire Line
+	1900 6000 1800 6000
+Wire Wire Line
+	1800 6000 1800 5900
+Wire Wire Line
+	1800 5900 1200 5900
+Connection ~ 1700 4300
+Connection ~ 1700 3700
+Connection ~ 1700 4800
+Connection ~ 1700 5300
+Connection ~ 1900 5800
 $EndSCHEMATC

Commit message: Introduce jumper for user IOREF
Parts:
- added JP18: Jumper_NC_Dual, symbol Jumper_NC_Dual
Connections:
- net labels added: IOREF_U
- wire segments 78 -> 84
Other:
- note added: "Selects 5/3V3 board variant\n(pull-up resistors, DHT power, ...)"

Commit message: Add pinhead for signals D+ and D- on USB connector
Parts:
- added J8: CONN_01X02, Pin_Headers:Pin_Header_Straight_1x02_Pitch2.54mm, symbol CONN_01X02
Connections:
- net labels added: D+, D-
- wire segments 84 -> 87
- no-connect marks 5 -> 3
Other:
- moved on the sheet: JP9

Commit message: Add ESP32-DevKitC to the schematics
Parts:
- added U3: ESP32-DEVKIT-C, yaqwsx:ESP32-DEVKIT-C, symbol ESP32-DEVKIT-C
Connections:
- wire segments 87 -> 91
- no-connect marks 3 -> 13
Other:
- note added: "ESP32 - boot1"
- note added: "ESP32 - boot2"
- moved on the sheet: JP16, JP4, PIEIZO1, R7, U1, U2

Commit message: Change LED resistors from 150R to 220R
Parts:
- R16, R17, R18, R5, R6, R7, R8, R9: value 150R -> 220R
Changed lines of the file:
@@
 P 9850 2650
 F 0 "R16" V 9930 2650 50  0000 C CNN
-F 1 "150R" V 9850 2650 50  0000 C CNN
+F 1 "220R" V 9850 2650 50  0000 C CNN
 F 2 "Resistors_SMD:R_1206_HandSoldering" H 9850 2650 50  0001 C CNN
 F 3 "" H 9850 2650 50  0000 C CNN
@@
 P 10050 2650
 F 0 "R17" V 10130 2650 50  0000 C CNN
-F 1 "150R" V 10050 2650 50  0000 C CNN
+F 1 "220R" V 10050 2650 50  0000 C CNN
 F 2 "Resistors_SMD:R_1206_HandSoldering" H 10050 2650 50  0001 C CNN
 F 3 "" H 10050 2650 50  0000 C CNN
@@
 P 10250 2650
 F 0 "R18" V 10330 2650 50  0000 C CNN
-F 1 "150R" V 10250 2650 50  0000 C CNN
+F 1 "220R" V 10250 2650 50  0000 C CNN
 F 2 "Resistors_SMD:R_1206_HandSoldering" H 10250 2650 50  0001 C CNN
 F 3 "" H 10250 2650 50  0000 C CNN
@@
 P 6700 3250
 F 0 "R8" V 6780 3250 50  0000 C CNN
-F 1 "150R" V 6700 3250 50  0000 C CNN
+F 1 "220R" V 6700 3250 50  0000 C CNN
 F 2 "Resistors_SMD:R_1206_HandSoldering" H 6700 3250 50  0001 C CNN
 F 3 "" H 6700 3250 50  0000 C CNN
@@
 P 6700 3600
 F 0 "R9" V 6780 3600 50  0000 C CNN
-F 1 "150R" V 6700 3600 50  0000 C CNN
+F 1 "220R" V 6700 3600 50  0000 C CNN
 F 2 "Resistors_SMD:R_1206_HandSoldering" H 6700 3600 50  0001 C CNN
 F 3 "" H 6700 3600 50  0000 C CNN
@@
 P 6700 3950
 F 0 "R5" V 6780 3950 50  0000 C CNN
-F 1 "150R" V 6700 3950 50  0000 C CNN
+F 1 "220R" V 6700 3950 50  0000 C CNN
 F 2 "Resistors_SMD:R_1206_HandSoldering" H 6700 3950 50  0001 C CNN
 F 3 "" H 6700 3950 50  0000 C CNN
@@
 P 6700 4300
 F 0 "R6" V 6780 4300 50  0000 C CNN
-F 1 "150R" V 6700 4300 50  0000 C CNN
+F 1 "220R" V 6700 4300 50  0000 C CNN
 F 2 "Resistors_SMD:R_1206_HandSoldering" H 6700 4300 50  0001 C CNN
 F 3 "" H 6700 4300 50  0000 C CNN
@@
 P 1100 1750
 F 0 "R7" V 1180 1750 50  0000 C CNN
-F 1 "150R" V 1100 1750 50  0000 C CNN
+F 1 "220R" V 1100 1750 50  0000 C CNN
 F 2 "Resistors_SMD:R_1206_HandSoldering" H 1100 1750 50  0001 C CNN
 F 3 "" H 1100 1750 50  0000 C CNN

Commit message: My rework
Parts:
- added J9: SPI, Pin_Headers:Pin_Header_Straight_1x04_Pitch2.54mm, symbol Connector_Generic:Conn_01x04
- added R26, R27: 3k3, Resistors_SMD:R_1206_HandSoldering, symbol Device:R
- C1, C2, C3: value 100n -> 10n; symbol C-RESCUE-robotarna_arduino -> Device:C
- C4, C5, C6, C7, C8: value C_Small -> 10 μF; symbol C_Small -> ArduinoLearningKitStarter-rescue:C_Small
- DHT11: footprint Pin_Headers:Pin_Header_Straight_1x04 -> Pin_Headers:Pin_Header_Straight_1x04_Pitch2.54mm; symbol CONN_01X04 -> ArduinoLearningKitStarter-rescue:Conn_01x04
- J1: symbol USB_OTG -> Connector:USB_B_Micro
- J2, J4: footprint yaqwsx:Pin_Header_Straight_1x08_circle -> Pin_Headers:Pin_Header_Straight_1x08_Pitch2.54mm; symbol CONN_01X08 -> Connector_Generic:Conn_01x08
- J3: footprint yaqwsx:Pin_Header_Straight_1x06_circle -> Pin_Headers:Pin_Header_Straight_1x06_Pitch2.54mm; symbol CONN_01X06 -> Connector_Generic:Conn_01x06
- J5: footprint yaqwsx:Pin_Header_Straight_1x10_circle -> Pin_Headers:Pin_Header_Straight_1x10_Pitch2.54mm; symbol CONN_01X10 -> Connector_Generic:Conn_01x10
- J6: footprint Pin_Headers:Pin_Header_Straight_1x04 -> Pin_Headers:Pin_Header_Angled_1x04_Pitch2.54mm; symbol CONN_01X04 -> Connector_Generic:Conn_01x04
- J7: symbol CONN_01X04 -> Connector_Generic:Conn_01x04
- J8: symbol CONN_01X02 -> Connector_Generic:Conn_01x02
- JP1, JP10, JP11, JP12, JP13, JP14, JP15, JP16, JP17, JP2, JP3, JP4, JP5, JP6, JP7, JP8, JP9: symbol Jumper_NC_Small -> Device:Jumper_NC_Small
- JP18: footprint (none) -> Pin_Headers:Pin_Header_Angled_1x03_Pitch2.54mm; symbol Jumper_NC_Dual -> Device:Jumper_NC_Dual
- L_B1, L_G1, L_R1, L_Y1: footprint LEDs:LED-5MM -> LEDs:LED_D5.0mm; symbol LED-RESCUE-robotarna_arduino -> Device:LED
- L_RGB1: footprint LEDs:LED-RGB-5MM_Common_Cathode -> LEDs:LED_D5.0mm-4; symbol LED_RCBG-RESCUE-robotarna_arduino -> Device:LED_RCBG
- PHOTO1: symbol Photores -> Device:R_PHOTO
- PIEZO1: renamed from PIEIZO1; symbol PIEZO -> yaqwsx:PIEZO
- R1, R10, R11, R12, R13, R14, R15, R16, R17, R18, R19, R2, R20, R21, R22, R23, R24, R25, R3, R4, R5, R6, R7, R8, R9: symbol R-RESCUE-robotarna_arduino -> Device:R
- RV1, RV2: footprint Potentiometers:RV09 -> yaqwsx:RV09; symbol POT-RESCUE-robotarna_arduino -> Device:R_POT
- S1, S2, S3, S4, S5: symbol CONN_01X03 -> Connector_Generic:Conn_01x03
- SW1, SW2, SW3: footprint Buttons_Switches_ThroughHole:SW_PUSH_6mm -> Buttons_Switches_THT:SW_PUSH_6mm; symbol SW_PUSH -> Switch:SW_Push
- U1: symbol arduino_nano -> yaqwsx:arduino_nano
- U2: symbol arduino_uno -> yaqwsx:arduino_uno
- U3: symbol ESP32-DEVKIT-C -> yaqwsx:ESP32-DEVKIT-C
Connections:
- net labels added: SCL, SDA
- wire segments 91 -> 194
Other:
- moved on the sheet: JP1, JP13, JP14, JP15, JP2, JP3, JP4, JP9, PIEZO1, R1, R16, R17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
