File: ArduinoLearningKitStarter.sch (KiCad schematic (older format))
At the start: 83 parts, among them J1 USB_OTG, J2 CONN_01X08, J3 CONN_01X06, J4 CONN_01X08, J5 CONN_01X10, J6 CONN_01X04, J7 CONN_01X04, J8 CONN_01X02, J9 SPI, SW1 SW_PUSH, SW2 SW_PUSH, SW3 SW_PUSH, U1 arduino_nano, U2 arduino_uno, U3 ESP32-DEVKIT-C

Commit message: Fix schematic libraries
Parts:
- C4, C5, C6, C7, C8: symbol ArduinoLearningKitStarter-rescue:C_Small -> ArduinoLearningKitStarter:C_Small
- DHT11: symbol ArduinoLearningKitStarter-rescue:Conn_01x04 -> ArduinoLearningKitStarter:Conn_01x04
- PIEZO1: symbol yaqwsx:PIEZO -> ArduinoLearningKitStarter:PIEZO-yaqwsx
- U1: symbol yaqwsx:arduino_nano -> ArduinoLearningKitStarter:arduino_nano-yaqwsx
- U2: symbol yaqwsx:arduino_uno -> ArduinoLearningKitStarter:arduino_uno-yaqwsx
- U3: symbol yaqwsx:ESP32-DEVKIT-C -> ArduinoLearningKitStarter:ESP32-DEVKIT-C-yaqwsx
Changed lines of the file:
@@
 EESchema Schematic File Version 4
-LIBS:ArduinoLearningKitStarter-cache
 EELAYER 26 0
 EELAYER END
@@
 $EndDescr
 $Comp
-L yaqwsx:arduino_nano U1
+L ArduinoLearningKitStarter:arduino_nano-yaqwsx U1
 U 1 1 57E2ED37
 P 6100 1650
@@
 $EndComp
 $Comp
-L yaqwsx:arduino_uno U2
+L ArduinoLearningKitStarter:arduino_uno-yaqwsx U2
 U 1 1 57E2EE30
 P 8700 1700
@@
 D0
 $Comp
-L ArduinoLearningKitStarter-rescue:+3V3 #PWR01
+L ArduinoLearningKitStarter:+3V3 #PWR01
 U 1 1 57E2F0DE
 P 4850 1050
@@
 $EndComp
 $Comp
-L ArduinoLearningKitStarter-rescue:+3V3 #PWR02
+L ArduinoLearningKitStarter:+3V3 #PWR02
 U 1 1 57E2F0F6
 P 7800 1500
@@
 $EndComp
 $Comp
-L ArduinoLearningKitStarter-rescue:+5V #PWR03
+L ArduinoLearningKitStarter:+5V #PWR03
 U 1 1 57E2F11D
 P 5050 2050
@@
 $EndComp
 $Comp
-L ArduinoLearningKitStarter-rescue:GND #PWR04
+L ArduinoLearningKitStarter:GND #PWR04
 U 1 1 57E2F135
 P 5050 2250
@@
 $EndComp
 $Comp
-L ArduinoLearningKitStarter-rescue:VCC #PWR05
+L ArduinoLearningKitStarter:VCC #PWR05
 U 1 1 57E2F14D
 P 5050 2350
@@
 $EndComp
 $Comp
-L ArduinoLearningKitStarter-rescue:GND #PWR06
+L ArduinoLearningKitStarter:GND #PWR06
 U 1 1 57E2F1D1
 P 7100 2050
@@
 $EndComp
 $Comp
-L ArduinoLearningKitStarter-rescue:GND #PWR07
+L ArduinoLearningKitStarter:GND #PWR07
 U 1 1 57E2F21B
 P 7950 1700
@@
 $EndComp
 $Comp
-L ArduinoLearningKitStarter-rescue:GND #PWR08
+L ArduinoLearningKitStarter:GND #PWR08
 U 1 1 57E2F238
 P 9750 1100
@@
 $EndComp
 $Comp
-L ArduinoLearningKitStarter-rescue:+5V #PWR09
+L ArduinoLearningKitStarter:+5V #PWR09
 U 1 1 57E2F25B
 P 7800 1600
@@
 $EndComp
 $Comp
-L ArduinoLearningKitStarter-rescue:VCC #PWR010
+L ArduinoLearningKitStarter:VCC #PWR010
 U 1 1 57E2F27C
 P 7800 1900
@@
 D10
 $Comp
-L ArduinoLearningKitStarter-rescue:GND #PWR011
+L ArduinoLearningKitStarter:GND #PWR011
 U 1 1 57E2F8C9
 P 9150 5300
@@
 $EndComp
 $Comp
-L ArduinoLearningKitStarter-rescue:GND #PWR012
+L ArduinoLearningKitStarter:GND #PWR012
 U 1 1 57E33F11
 P 6700 5100
@@
 $EndComp
 $Comp
-L ArduinoLearningKitStarter-rescue:GND #PWR013
+L ArduinoLearningKitStarter:GND #PWR013
 U 1 1 57E35660
 P 6950 3250
@@
 $EndComp
 $Comp
-L ArduinoLearningKitStarter-rescue:GND #PWR014
+L ArduinoLearningKitStarter:GND #PWR014
 U 1 1 57E35DEA
 P 6950 3600
@@
 $EndComp
 $Comp
-L ArduinoLearningKitStarter-rescue:GND #PWR015
+L ArduinoLearningKitStarter:GND #PWR015
 U 1 1 57E3661D
 P 6950 3950
@@
 $EndComp
 $Comp
-L ArduinoLearningKitStarter-rescue:GND #PWR016
+L ArduinoLearningKitStarter:GND #PWR016
 U 1 1 57E36640
 P 6950 4300
@@
 $EndComp
 $Comp
-L ArduinoLearningKitStarter-rescue:GND #PWR017
+L ArduinoLearningKitStarter:GND #PWR017
 U 1 1 57E3786D
 P 6450 7550
@@
 $EndComp
 $Comp
-L ArduinoLearningKitStarter-rescue:GND #PWR018
+L ArduinoLearningKitStarter:GND #PWR018
 U 1 1 57E39E55
 P 10700 2300
@@
 $EndComp
 $Comp
-L ArduinoLearningKitStarter-rescue:GND #PWR019
+L ArduinoLearningKitStarter:GND #PWR019
 U 1 1 57E4523D
 P 6700 5850
@@
 D3
 $Comp
-L ArduinoLearningKitStarter-rescue:GND #PWR020
+L ArduinoLearningKitStarter:GND #PWR020
 U 1 1 57E4799B
 P 9150 3500
@@
 D4
 $Comp
-L ArduinoLearningKitStarter-rescue:GND #PWR021
+L ArduinoLearningKitStarter:GND #PWR021
 U 1 1 57E47D6B
 P 9150 4300
@@
 $EndComp
 $Comp
-L ArduinoLearningKitStarter-rescue:Conn_01x04 DHT11
+L ArduinoLearningKitStarter:Conn_01x04 DHT11
 U 1 1 57E4A74C
 P 10650 3050
@@
 $EndComp
 $Comp
-L ArduinoLearningKitStarter-rescue:GND #PWR022
+L ArduinoLearningKitStarter:GND #PWR022
 U 1 1 57E4A971
 P 10450 3250
@@
 $EndComp
 $Comp
-L yaqwsx:PIEZO PIEZO1
+L ArduinoLearningKitStarter:PIEZO-yaqwsx PIEZO1
 U 1 1 57E2F3A6
 P 1100 2100
@@
 VCC_SERVO
 $Comp
-L ArduinoLearningKitStarter-rescue:GND #PWR023
+L ArduinoLearningKitStarter:GND #PWR023
 U 1 1 58C26AD7
 P 1250 3250
@@
 $EndComp
 $Comp
-L ArduinoLearningKitStarter-rescue:GND #PWR024
+L ArduinoLearningKitStarter:GND #PWR024
 U 1 1 58C26C94
 P 1250 3900
@@
 $EndComp
 $Comp
-L ArduinoLearningKitStarter-rescue:GND #PWR025
+L ArduinoLearningKitStarter:GND #PWR025
 U 1 1 58C26D59
 P 1250 4550
@@
 $EndComp
 $Comp
-L ArduinoLearningKitStarter-rescue:GND #PWR026
+L ArduinoLearningKitStarter:GND #PWR026
 U 1 1 58C26F92
 P 1250 5150
@@
 $EndComp
 $Comp
-L ArduinoLearningKitStarter-rescue:GND #PWR027
+L ArduinoLearningKitStarter:GND #PWR027
 U 1 1 58C2711B
 P 1250 5750
@@
 D10
 $Comp
-L ArduinoLearningKitStarter-rescue:GND #PWR028
+L ArduinoLearningKitStarter:GND #PWR028
 U 1 1 58C2A0F7
 P 1150 7250
@@
 $EndComp
 $Comp
-L ArduinoLearningKitStarter-rescue:+5V #PWR029
+L ArduinoLearningKitStarter:+5V #PWR029
 U 1 1 58C30598
 P 1800 6400
@@
 $EndComp
 $Comp
-L ArduinoLearningKitStarter-rescue:+5V #PWR030
+L ArduinoLearningKitStarter:+5V #PWR030
 U 1 1 58C30CE3
 P 4350 4100
@@
 $EndComp
 $Comp
-L ArduinoLearningKitStarter-rescue:GND #PWR031
+L ArduinoLearningKitStarter:GND #PWR031
 U 1 1 58C31560
 P 4350 4900
@@
 $EndComp
 $Comp
-L ArduinoLearningKitStarter-rescue:GND #PWR032
+L ArduinoLearningKitStarter:GND #PWR032
 U 1 1 58C319C6
 P 4350 5900
@@
 $EndComp
 $Comp
-L ArduinoLearningKitStarter-rescue:GND #PWR033
+L ArduinoLearningKitStarter:GND #PWR033
 U 1 1 58C326A3
 P 4350 7150
@@
 IOREF
 $Comp
-L ArduinoLearningKitStarter-rescue:GND #PWR034
+L ArduinoLearningKitStarter:GND #PWR034
 U 1 1 58C335CF
 P 4400 3400
@@
 IOREF
 $Comp
-L ArduinoLearningKitStarter-rescue:GND #PWR035
+L ArduinoLearningKitStarter:GND #PWR035
 U 1 1 58C33A9B
 P 4100 3600
@@
 $EndComp
 $Comp
-L ArduinoLearningKitStarter-rescue:+3V3 #PWR036
+L ArduinoLearningKitStarter:+3V3 #PWR036
 U 1 1 58C33C8A
 P 3900 3700
@@
 $EndComp
 $Comp
-L ArduinoLearningKitStarter-rescue:GND #PWR037
+L ArduinoLearningKitStarter:GND #PWR037
 U 1 1 58C39C30
 P 3200 6550
@@
 D1
 $Comp
-L ArduinoLearningKitStarter-rescue:GND #PWR038
+L ArduinoLearningKitStarter:GND #PWR038
 U 1 1 58C3D24F
 P 3350 5600
@@
 D2
 $Comp
-L ArduinoLearningKitStarter-rescue:C_Small C4
+L ArduinoLearningKitStarter:C_Small C4
 U 1 1 58DE66DE
 P 1600 3250
@@
 $EndComp
 $Comp
-L ArduinoLearningKitStarter-rescue:C_Small C5
+L ArduinoLearningKitStarter:C_Small C5
 U 1 1 58DE6B28
 P 1600 3900
@@
 $EndComp
 $Comp
-L ArduinoLearningKitStarter-rescue:C_Small C6
+L ArduinoLearningKitStarter:C_Small C6
 U 1 1 58DE6CDD
 P 1600 4550
@@
 $EndComp
 $Comp
-L ArduinoLearningKitStarter-rescue:C_Small C7
+L ArduinoLearningKitStarter:C_Small C7
 U 1 1 58DE7055
 P 1600 5150
@@
 $EndComp
 $Comp
-L ArduinoLearningKitStarter-rescue:C_Small C8
+L ArduinoLearningKitStarter:C_Small C8
 U 1 1 58DE720C
 P 1600 5750
@@
 IOREF_U
 $Comp
-L ArduinoLearningKitStarter-rescue:+5V #PWR039
+L ArduinoLearningKitStarter:+5V #PWR039
 U 1 1 590233A7
 P 9900 5250
@@
 $EndComp
 $Comp
-L ArduinoLearningKitStarter-rescue:+3V3 #PWR040
+L ArduinoLearningKitStarter:+3V3 #PWR040
 U 1 1 590237F3
 P 10750 5250
@@
 D-
 $Comp
-L yaqwsx:ESP32-DEVKIT-C U3
+L ArduinoLearningKitStarter:ESP32-DEVKIT-C-yaqwsx U3
 U 1 1 5914FD59
 P 2950 1850
@@
 $EndComp
 $Comp
-L ArduinoLearningKitStarter-rescue:+3V3 #PWR041
+L ArduinoLearningKitStarter:+3V3 #PWR041
 U 1 1 5914FF34
 P 2450 950
@@
 $EndComp
 $Comp
-L ArduinoLearningKitStarter-rescue:+5V #PWR042
+L ArduinoLearningKitStarter:+5V #PWR042
 U 1 1 59150129
 P 2450 2750
@@
 $EndComp
 $Comp
-L ArduinoLearningKitStarter-rescue:GND #PWR043
+L ArduinoLearningKitStarter:GND #PWR043
 U 1 1 5915031E
 P 3800 1550
@@
 $EndComp
 $Comp
-L ArduinoLearningKitStarter-rescue:GND #PWR044
+L ArduinoLearningKitStarter:GND #PWR044
 U 1 1 59150419
 P 2200 2250
@@
 $EndComp
 $Comp
-L ArduinoLearningKitStarter-rescue:GND #PWR045
+L ArduinoLearningKitStarter:GND #PWR045
 U 1 1 59150514
 P 3850 950
@@
 IOREF_U
 $Comp
-L ArduinoLearningKitStarter-rescue:GND #PWR0101
+L ArduinoLearningKitStarter:GND #PWR0101
 U 1 1 5BCC427E
 P 10550 4450
