File: ArduinoLearningKitStarter.sch (KiCad schematic (older format))
At the start: 87 parts, among them J1 USB_OTG, J10 DHT11, J2 CONN_01X08, J3 CONN_01X06, J4 CONN_01X08, J5 CONN_01X10, J6 I2C, J7 CONN_01X04, J8 CONN_01X02, J9 SPI, SW1 SW_PUSH, SW2 SW_PUSH, SW3 SW_PUSH, U1 arduino_nano, U2 arduino_uno, U3 ESP32-DEVKIT-C

Commit message: Remove Arduino holes, change photo footprint and add IOREF header
Parts:
- removed H1, H2, H3, H4: Arduino Uno Mounting, MountingHole:MountingHole_2.2mm_M2, symbol Mechanical:MountingHole
- J2, J4: footprint Connector_PinHeader_2.54mm:PinHeader_1x08_P2.54mm_Vertical -> Connector_PinHeader_2.54mm:PinHeader_2x08_P2.54mm_Vertical; symbol Connector_Generic:Conn_01x08 -> Connector_Generic:Conn_02x08_Odd_Even
- J3: footprint Connector_PinHeader_2.54mm:PinHeader_1x06_P2.54mm_Vertical -> Connector_PinHeader_2.54mm:PinHeader_2x06_P2.54mm_Vertical; symbol Connector_Generic:Conn_01x06 -> Connector_Generic:Conn_02x06_Odd_Even
- J5: footprint Connector_PinHeader_2.54mm:PinHeader_1x10_P2.54mm_Vertical -> Connector_PinHeader_2.54mm:PinHeader_2x10_P2.54mm_Vertical; symbol Connector_Generic:Conn_01x10 -> Connector_Generic:Conn_02x10_Odd_Even
- PHOTO1: footprint Resistors_ThroughHole:Resistor_Horizontal_RM7mm -> ALKS:PHOTO
Connections:
- net +3V3: no longer J2.4 (Pin_4)
- net +5V: no longer J2.5 (Pin_5), J2.6 (Pin_6), J2.7 (Pin_7), J2.8 (Pin_8)
- net GND: now also J2.11 (Pin_11), J2.13 (Pin_13), J2.15 (Pin_15), J2.5 (Pin_5), J2.7 (Pin_7), J2.9 (Pin_9), J3.11 (Pin_11), J3.7 (Pin_7), J3.9 (Pin_9), J4.11 (Pin_11), J4.13 (Pin_13), J4.15 (Pin_15), J4.9 (Pin_9), J5.11 (Pin_11), J5.13 (Pin_13), J5.15 (Pin_15), J5.17 (Pin_17), J5.19 (Pin_19); no longer J3.2 (Pin_2), J3.4 (Pin_4), J3.6 (Pin_6), J4.2 (Pin_2), J4.4 (Pin_4), J4.6 (Pin_6), J4.8 (Pin_8), J5.10 (Pin_10), J5.2 (Pin_2), J5.4 (Pin_4), J5.6 (Pin_6), J5.8 (Pin_8)
- net IOREF: now also J2.10 (Pin_10), J2.12 (Pin_12), J2.14 (Pin_14), J2.16 (Pin_16), J2.4 (Pin_4), J2.6 (Pin_6), J2.8 (Pin_8), J3.10 (Pin_10), J3.12 (Pin_12), J3.2 (Pin_2), J3.4 (Pin_4), J3.6 (Pin_6), J3.8 (Pin_8), J4.10 (Pin_10), J4.12 (Pin_12), J4.14 (Pin_14), J4.16 (Pin_16), J4.2 (Pin_2), J4.4 (Pin_4), J4.6 (Pin_6), J4.8 (Pin_8), J5.10 (Pin_10), J5.12 (Pin_12), J5.14 (Pin_14), J5.16 (Pin_16), J5.18 (Pin_18), J5.2 (Pin_2), J5.20 (Pin_20), J5.4 (Pin_4), J5.6 (Pin_6), J5.8 (Pin_8)
Other:
- moved on the sheet: J7, R3
